Commit message: Update description package
clhero_description coincide ahora con el robot real. Incluye la RealSense y las patas se mueven correctamente en RViz

File: clhero_description/robots/clhero.robot.xacro (robot description, xacro)
@@ -69,5 +69,5 @@
 </hokuyo_sensor-->
 <sensor_d435 parent="base_link">
-    <origin xyz="0.27 0 -0.01" rpy="0 0 0"/>
+    <origin xyz="0.27 0 -0.01" rpy="0 0 $(pi)"/>
 </sensor_d435>
 </robot>

File: clhero_description/robots/clhero.urdf.xacro (robot description, xacro)
@@ -19,34 +19,34 @@
 <!-- Instanciacion de las patas dentro de la descripcion del robot -->
 <pata_c name="motor_1" parent_link="base_link" right="0">
-    <origin xyz="${-235/1000} ${233/1000} ${0/1000}" rpy="0 0 0"/>
+    <origin xyz="${-235/1000} ${298/1000} ${0/1000}" rpy="0 0 ${pi}"/>
 </pata_c>
 <pata_c name="motor_2" parent_link="base_link" right="1">
-    <origin xyz="${-235/1000} ${-233/1000} ${0/1000}" rpy="0 0 0"/>
+    <origin xyz="${-235/1000} ${-253/1000} ${0/1000}" rpy="0 0 ${pi}"/>
 </pata_c>
 <pata_c name="motor_3" parent_link="base_link" right="0">
-    <origin xyz="${0/1000} ${289/1000} ${0/1000}" rpy="0 0 0"/>
+    <origin xyz="${0/1000} ${354/1000} ${0/1000}" rpy="0 0 ${pi}"/>
 </pata_c>
 <pata_c name="motor_4" parent_link="base_link" right="1">
-    <origin xyz="${0/1000} ${-289/1000} ${0/1000}" rpy="0 0 0"/>
+    <origin xyz="${0/1000} ${-303/1000} ${0/1000}" rpy="0 0 ${pi}"/>
 </pata_c>
 <pata_c name="motor_5" parent_link="base_link" right="0">
-    <origin xyz="${235/1000} ${233/1000} ${0/1000}" rpy="0 0 0"/>
+    <origin xyz="${235/1000} ${298/1000} ${0/1000}" rpy="0 0 ${pi}"/>
 </pata_c>
 <pata_c name="motor_6" parent_link="base_link" right="1">
-    <origin xyz="${235/1000} ${-233/1000} ${0/1000}" rpy="0 0 0"/>
+    <origin xyz="${235/1000} ${-253/1000} ${0/1000}" rpy="0 0 ${pi}"/>
 </pata_c>
 <!-- Instanciacion de la camara kinect dentro de la descripcion del robot -->
 <!--kinect_camera name="kin" parent_link="base_link">
-    <origin xyz="${300/1000} ${0/1000} ${0/1000}" rpy="0 0 0"/>
+    <origin xyz="${300/1000} ${0/1000} ${0/1000}" rpy="0 0 ${pi/2}"/>
 </kinect_camera-->
 <!-- Instanciacion de la IMU dentro de la descripcion del robot -->
 <!--imu name="imu1" parent_link="base_link">
-    <origin xyz="${0/1000} ${0/1000} ${40/1000}" rpy="0 0 0"/>
+    <origin xyz="${0/1000} ${0/1000} ${40/1000}" rpy="0 0 ${pi/2}"/>
 </imu-->
 <!--hokuyo_sensor sensor_name="hokuyo" parent_name="base_link">
-    <origin xyz="${300/1000} 0 0" rpy="0 0 0"/>
+    <origin xyz="${300/1000} 0 0" rpy="0 0 ${pi/2}"/>
 </hokuyo_sensor-->
 <sensor_d435 parent="base_link">
-    <origin xyz="0.27 0 -0.01" rpy="0 0 0"/>
+    <origin xyz="-0.27 0 -0.01" rpy="0 0 ${pi}"/>
 </sensor_d435>
 </robot>

File: clhero_description/urdf/base.xacro (robot description, xacro)
@@ -49,5 +49,6 @@
     <parent link="base_footprint"/>
     <child link="base_link"/>
-    <origin xyz="0 0 ${w_radius*2}" rpy="0 0 0"/>
+    <!--origin xyz="0 0 ${w_radius*2}" rpy="0 0 0"/-->
+    <origin xyz="0 0 ${0.04}" rpy="0 0 0"/>
 </joint>
 </robot>

File: clhero_description/urdf/base_cinta.xacro (robot description, xacro)
@@ -29,5 +29,5 @@
         <origin xyz="0 0 0.38" rpy="0 0 ${pi/2}"/>
         <geometry>
-            <mesh filename="package://hexapodo_description/meshes/cinta_barreras.stl" scale="0.01 0.01 0.01"/>
+            <mesh filename="package://clhero_description/meshes/cinta_barreras.stl" scale="0.01 0.01 0.01"/>
         </geometry>
         <material name="base_link_material">
@@ -44,5 +44,5 @@
         <origin xyz="0 0 0.358" rpy="0 0 0"/>
         <geometry>
-            <mesh filename="package://hexapodo_description/meshes/cinta_barreras.stl" scale="0.01 0.01 0.01"/>
+            <mesh filename="package://clhero_description/meshes/cinta_barreras.stl" scale="0.01 0.01 0.01"/>
         </geometry>
     </collision-->
@@ -65,5 +65,5 @@
         <origin xyz="${-300/1e3} 0 0.0" rpy="${pi/2} 0 ${pi/2}"/>
         <geometry>
-            <mesh filename="package://hexapodo_description/meshes/chassis.stl" scale="0.001 0.001 0.001"/>
+            <mesh filename="package://clhero_description/meshes/chassis.stl" scale="0.001 0.001 0.001"/>
         </geometry>
         <material name="chassis_material">
@@ -74,5 +74,5 @@
         <origin xyz="${-300/1e3} 0 0.0" rpy="${pi/2} 0 ${pi/2}"/>
         <geometry>
-            <mesh filename="package://hexapodo_description/meshes/chassis.stl" scale="0.001 0.001 0.001"/>
+            <mesh filename="package://clhero_description/meshes/chassis.stl" scale="0.001 0.001 0.001"/>
         </geometry>
     </collision>

File: clhero_description/urdf/pata_c.xacro (robot description, xacro)
@@ -30,11 +30,11 @@
         <visual>
             <xacro:if value="${right == 1}">
-                <origin xyz="0 0 0" rpy="${pi/2} 0 0"/>
+                <origin xyz="0 0 0" rpy="${pi/2} 0 ${pi}"/>
             </xacro:if>
             <xacro:if value="${right == 0}">
-                <origin xyz="0 0.05 0" rpy="${pi/2} 0 0"/>
+                <origin xyz="0 0.05 0" rpy="${pi/2} 0 ${pi}"/>
             </xacro:if>
             <geometry>
-                <mesh filename="package://hexapodo_description/meshes/pvc.stl" scale="0.001 0.001 0.001"/>
+                <mesh filename="package://clhero_description/meshes/clegs_80.stl" scale="0.001 0.001 0.001"/>
             </geometry>
             <material name="Grey">
@@ -50,5 +50,5 @@
             </xacro:if>
             <geometry>
-                <mesh filename="package://hexapodo_description/meshes/pvc.stl" scale="0.001 0.001 0.001"/>
+                <mesh filename="package://clhero_description/meshes/clegs_80.stl" scale="0.001 0.001 0.001"/>
             </geometry>
             <surface>

File: clhero_description/urdf/pata_c_cinta.xacro (robot description, xacro)
@@ -30,5 +30,5 @@
             </xacro:if>
             <geometry>
-                <mesh filename="package://hexapodo_description/meshes/pvc.stl" scale="0.001 0.001 0.001"/>
+                <mesh filename="package://clhero_description/meshes/clegs_80.stl" scale="0.001 0.001 0.001"/>
             </geometry>
             <material name="Grey">
@@ -44,5 +44,5 @@
             </xacro:if>
             <geometry>
-                <mesh filename="package://hexapodo_description/meshes/pvc.stl" scale="0.001 0.001 0.001"/>
+                <mesh filename="package://clhero_description/meshes/clegs_80.stl" scale="0.001 0.001 0.001"/>
             </geometry>
         </collision>

Commit message: github backup

File: clhero_description/robots/clhero.robot.xacro (robot description, xacro)
@@ -69,5 +69,5 @@
 </hokuyo_sensor-->
 <sensor_d435 parent="base_link">
-    <origin xyz="0.27 0 -0.01" rpy="0 0 $(pi)"/>
+    <origin xyz="0.27 0 -0.01" rpy="0 0 0"/>
 </sensor_d435>
 </robot>

File: clhero_description/robots/clhero.urdf.xacro (robot description, xacro)
@@ -7,8 +7,13 @@
 <xacro:include filename="$(find clhero_description)/urdf/pata_c.xacro"/>
 <xacro:include filename="$(find clhero_description)/urdf/base.xacro"/>
-<!--xacro:include filename="$(find clhero_description)/urdf/sensores/kinect_camera.xacro"/>
+<!--xacro:include filename="$(find clhero_description)/urdf/sensores/kinect_camera.xacro"/-->
 <xacro:include filename="$(find clhero_description)/urdf/sensores/imu.xacro"/>
-<xacro:include filename="$(find clhero_description)/urdf/sensores/hokuyo_sensor.xacro"/-->
-<xacro:include filename="$(find realsense2_description)/urdf/_d435.urdf.xacro"/>
+<!--xacro:include filename="$(find clhero_description)/urdf/sensores/hokuyo_sensor.xacro"/-->
+<!--xacro:include filename="$(find realsense_gazebo_plugin)/urdf/realsense-RS200.macro.xacro" /-->
+<!-- Camara stereo-->
+<xacro:include filename="$(find clhero_description)/urdf/sensores/component_snippets.xacro"/>
+<!--xacro:include filename="$(find realsense2_description)/urdf/_d435.urdf.xacro"/-->
+<!-- RealSense simulada -->
+<!--xacro:include filename="$(find realsense_gazebo_plugin)/urdf/realsense-RS200.macro.xacro"/-->
 <!-- Declaracion del plugin gazebo_ros_control -->
 <gazebo>
@@ -40,13 +45,22 @@
     <origin xyz="${300/1000} ${0/1000} ${0/1000}" rpy="0 0 ${pi/2}"/>
 </kinect_camera-->
-<!-- Instanciacion de la IMU dentro de la descripcion del robot -->
-<!--imu name="imu1" parent_link="base_link">
-    <origin xyz="${0/1000} ${0/1000} ${40/1000}" rpy="0 0 ${pi/2}"/>
-</imu-->
-<!--hokuyo_sensor sensor_name="hokuyo" parent_name="base_link">
-    <origin xyz="${300/1000} 0 0" rpy="0 0 ${pi/2}"/>
-</hokuyo_sensor-->
-<sensor_d435 parent="base_link">
-    <origin xyz="-0.27 0 -0.01" rpy="0 0 ${pi}"/>
-</sensor_d435>
+<!-- IMU -->
+<imu name="imu" parent_link="base_link">
+    <origin xyz="${0/1000} ${0/1000} ${40/1000}" rpy="0 0 ${pi}"/>
+</imu>
+<hokuyo_sensor sensor_name="clhero" parent_name="base_link">
+    <origin xyz="${-300/1000} 0 ${100/1000}" rpy="0 0 ${pi}"/>
+</hokuyo_sensor>
+<!--sensor_d435 parent="base_link">
+    <origin xyz="0.27 0 -0.01" rpy="0 0 ${pi/2}"/>
+</sensor_d435-->
+<!-- Camara estereo -->
+<xacro:vi_sensor_macro
+    namespace="/clhero"
+    parent_link="base_link"
+    enable_cameras="true"
+    enable_depth="true"
+    enable_ground_truth="false">
+    <origin xyz="-0.27 0.0 0.0" rpy="0 ${0} ${pi}" />
+</xacro:vi_sensor_macro>
 </robot>

File: clhero_description/urdf/base.xacro (robot description, xacro)
@@ -50,5 +50,5 @@
     <child link="base_link"/>
     <!--origin xyz="0 0 ${w_radius*2}" rpy="0 0 0"/-->
-    <origin xyz="0 0 ${0.04}" rpy="0 0 0"/>
+    <origin xyz="0 0 ${0.04}" rpy="0 0 ${pi}"/>
 </joint>
 </robot>

File: clhero_description/urdf/pata_c.xacro (robot description, xacro)
@@ -1,7 +1,7 @@
 <?xml version="1.0" ?>
 <robot name="pata_c" xmlns:xacro="http://ros.org/wiki/xacro">
-<!--xacro:property name="motor_reduction"  value="${529.0/16}"/-->
-<xacro:property name="motor_reduction"  value="${1}"/>
-<xacro:property name="motor_max_effort" value="${20}"/>
+<xacro:property name="motor_reduction"  value="${529.0/16}"/>
+<!--xacro:property name="motor_reduction"  value="${1}"/-->
+<xacro:property name="motor_max_effort" value="${100}"/>
 <!--xacro:property name="motor_max_effort" value="${12}"/-->
 <xacro:property name="motor_max_rev"    value="${1256.637/motor_reduction}"/>
@@ -44,8 +44,8 @@
         <collision>
             <xacro:if value="${right == 1}">
-                <origin xyz="0 0 0" rpy="${pi/2} 0 0"/>
+                <origin xyz="0 0 0" rpy="${pi/2} 0 ${pi}"/>
             </xacro:if>
             <xacro:if value="${right == 0}">
-                <origin xyz="0 0.05 0" rpy="${pi/2} 0 0"/>
+                <origin xyz="0 0.05 0" rpy="${pi/2} 0 ${pi}"/>
             </xacro:if>
             <geometry>
@@ -91,10 +91,24 @@
     <!--*******************************************************************************************-->
     <gazebo reference="${name}_pata_c_link">
-        <mu1 value="100000.0"/>
-        <mu2 value="100000.0"/>
+        <mu1 value="1"/>
+        <mu2 value="1"/>
         <kp  value="10000000.0" />
         <kd  value="1.0" />
         <fdir1 value="1 0 0"/>
         <material>Gazebo/Grey</material>
+        <surface>
+            <friction>
+                <torsional>
+                    <coefficient>10</coefficient>
+                    <use_patch_radius>true</use_patch_radius>
+                    <surface_radius>0.05</surface_radius>
+                    <patch_radius>0.01</patch_radius>
+                </torsional>
+            </friction>
+            <contact>
+                <poissons_ratio>0.5</poissons_ratio>
+                <elastic_modulus>1e8</elastic_modulus>
+            </contact>
+        </surface>
     </gazebo>
 </xacro:macro>

File: clhero_description/urdf/sensores/hokuyo_sensor.xacro (robot description, xacro)
@@ -57,5 +57,5 @@
             </ray>
             <plugin name="gazebo_ros_head_hokuyo_controller" filename="libgazebo_ros_laser.so">
-              <topicName>/robotest/laser/scan</topicName>
+              <topicName>/clhero/laser/scan</topicName>
               <frameName>${sensor_name}_hokuyo_base</frameName>
             </plugin>
